Commit message: lab-7

File: beginner_tutorials/urdf/my_robot.urdf (robot description, URDF)
Before this commit: robot materials, 4 links, 3 joints
Links:
- link link_3: geometry visual box size=0.24 0.045 0.045
Joints:
- joint base_to_link_2: limit lower=-1 upper=1 effort=30 velocity=1 -> lower=-1 upper=1 effort=30 velocity=1.0; origin xyz=0.03 0 0.1 -> xyz=0 0 0.098 rpy=0 0 0
- joint base_to_link_3: limit lower=-1 upper=-1 effort=30 velocity=1.0 -> lower=-1 upper=1 effort=30 velocity=1.0; origin xyz=0.08 0 0.134 rpy=0 0 0 -> xyz=0.15 0 0.18 rpy=0 0 0
